Commit message: RobotROS.urdf

File: robot_ros/urdf/RobotROS.urdf (robot description, URDF)
Before this commit: robot RobotROS, 6 links, 5 joints
Links:
- added link lidar_link, mass 0.1; collision cylinder length=0.05 radius=0.03; visual cylinder length=0.02 radius=0.03
- link base_link: geometry collision mesh filename=package://robot_ros/meshes/base_link2.dae scale=1 1 1; visual mesh filename=package://robot_ros/meshes/base_link2.dae scale=1 1 1
Joints:
- added joint lidar_joint: type fixed, parent base_link, child lidar_link, origin xyz=0 0 0.12 rpy=0 0 0
- joint base_footprint_joint: origin xyz=0 0 0 rpy=0 0 0 -> xyz=0 0 0.05 rpy=0 0 0
